File: main/main.kicad_sch (KiCad schematic)
At the start: 158 parts, among them SW1 SW_Push, SW10 SW_Push, SW11 SW_Push, SW12 SW_Push, SW13 SW_Push, SW14 SW_Push, SW15 SW_Push, SW16 SW_Push, SW17 SW_Push, SW18 SW_Push, SW19 SW_Push, SW2 SW_Push, SW20 SW_Push, SW21 SW_Push, SW22 SW_Push, SW23 SW_Push, SW24 SW_Push, SW25 SW_Push, SW26 SW_Push, SW27 SW_Push, SW28 SW_Push, SW29 SW_Push, SW3 SW_Push, SW31 SW_Push, SW32 SW_Push, SW33 SW_Push, SW34 SW_Push, SW35 SW_Push, SW36 SW_Push, SW37 SW_Push, SW38 SW_Push, SW39 SW_Push, SW4 SW_Push, SW40 SW_Push, SW41 SW_Push, SW42 SW_Push, SW43 SW_Push, SW44 SW_Push, SW45 SW_Push, SW46 SW_Push, SW47 SW_Push, SW48 SW_Push, SW49 SW_Push, SW5 SW_Push, SW50 SW_Push, SW51 SW_Push, SW52 SW_Push, SW53 SW_Push, SW54 SW_Push, SW55 SW_Push, SW56 SW_Push, SW57 SW_Push, SW58 SW_Push, SW59 SW_Push, SW6 SW_Push, SW60 SW_Push, SW61 SW_Push, SW62 SW_Push, SW63 SW_Push, SW64 SW_Push, SW65 SW_Push, SW66 SW_Push, SW67 SW_Push, SW68 SW_Push, SW69 SW_Push, SW7 SW_Push, SW70 SW_Push, SW71 SW_Push, SW72 SW_Push, SW73 SW_Push, SW74 SW_Push, SW75 SW_Push, SW76 SW_Push, SW8 SW_Push, SW9 SW_Push

Commit message: マイコンのシンボルとフットプリント完成？ 次はマイコンとフットプリントの回路図を作成
Parts:
- removed L1, L2, L3, L4, L5, L6: SK6812MINI, kbd_Parts:LED_SK6812MINI-E_BL, symbol Salicylic_kbd:LED_SK6812MINI-E
- removed SW1 (x2): SW_Push, symbol Switch:SW_Push
- added D77: D, symbol Device:D
- added SW1, SW30, SW77: SW_Push, symbol Switch:SW_Push
- added U1: MCP23017_SO, Package_SO:SOIC-28W_7.5x17.9mm_P1.27mm, symbol Interface_Expansion:MCP23017_SO
- added U2: AE-NRF52840, Original:AE-NRF52840_DIP32_700mil, symbol Original:AE-NRF52840
Connections:
- net LED: now also U2.9 (D13)
- net at D1.2 (A): now also SW1.2
- net at D30.2 (A): now also SW30.2
- removed net col0: SW15.1, SW29.1, SW42.1, SW43.1, SW57.1
- removed net col1: SW16.1, SW2.1, SW44.1, SW55.1, SW58.1
- removed net col10: SW11.1, SW25.1, SW39.1, SW53.1, SW73.1
- removed net col11: SW12.1, SW26.1, SW40.1, SW54.1, SW74.1
- removed net col12: SW13.1, SW27.1, SW41.1, SW75.1
- removed net col13: SW14.1, SW28.1, SW76.1
- removed net col2: SW17.1, SW3.1, SW31.1, SW45.1, SW56.1, SW59.1
- removed net col3: SW18.1, SW32.1, SW4.1, SW46.1, SW60.1, SW66.1
- removed net col4: SW19.1, SW33.1, SW47.1, SW5.1, SW61.1, SW67.1
- removed net col5: SW20.1, SW34.1, SW48.1, SW6.1, SW62.1, SW68.1
- removed net col6: SW21.1, SW35.1, SW49.1, SW63.1, SW69.1, SW7.1
- removed net col7: SW22.1, SW36.1, SW50.1, SW64.1, SW70.1, SW8.1
- removed net col8: SW23.1, SW37.1, SW51.1, SW65.1, SW71.1, SW9.1
- removed net col9: SW10.1, SW24.1, SW38.1, SW52.1, SW72.1
- removed net row0: D1.1 (K), D10.1 (K), D11.1 (K), D12.1 (K), D13.1 (K), D14.1 (K), D2.1 (K), D3.1 (K), D4.1 (K), D5.1 (K), D6.1 (K), D7.1 (K), D8.1 (K), D9.1 (K)
- removed net row1: D15.1 (K), D16.1 (K), D17.1 (K), D18.1 (K), D19.1 (K), D20.1 (K), D21.1 (K), D22.1 (K), D23.1 (K), D24.1 (K), D25.1 (K), D26.1 (K), D27.1 (K), D28.1 (K)
- removed net row2: D42.1 (K), D55.1 (K), D56.1 (K), D66.1 (K), D67.1 (K), D68.1 (K), D69.1 (K), D70.1 (K), D71.1 (K), D72.1 (K), D73.1 (K), D74.1 (K), D75.1 (K), D76.1 (K)
- removed net row3: D29.1 (K), D30.1 (K), D31.1 (K), D32.1 (K), D33.1 (K), D34.1 (K), D35.1 (K), D36.1 (K), D37.1 (K), D38.1 (K), D39.1 (K), D40.1 (K), D41.1 (K)
- removed net row4: D43.1 (K), D44.1 (K), D45.1 (K), D46.1 (K), D47.1 (K), D48.1 (K), D49.1 (K), D50.1 (K), D51.1 (K), D52.1 (K), D53.1 (K), D54.1 (K)
- removed net row5: D57.1 (K), D58.1 (K), D59.1 (K), D60.1 (K), D61.1 (K), D62.1 (K), D63.1 (K), D64.1 (K), D65.1 (K)
- new net: U1.10 (VSS), U2.20 (GND)
- new net: U1.9 (VDD), U2.18 (+3V3)
- new net: D77.2 (A), SW77.2
- new net c0: SW1.1, SW2.1, SW3.1, SW4.1, SW5.1, SW6.1, U1.1 (GPB0)
- new net c1: SW10.1, SW11.1, SW12.1, SW7.1, SW8.1, SW9.1, U1.2 (GPB1)
- new net c10: SW61.1, SW62.1, SW63.1, SW64.1, SW65.1, U1.24 (GPA3)
- new net c11: SW66.1, SW67.1, SW68.1, SW69.1, SW70.1, U1.25 (GPA4)
- new net c12: SW71.1, SW72.1, SW73.1, SW74.1, U1.26 (GPA5)
- new net c13: SW75.1, SW76.1, SW77.1, U1.27 (GPA6)
- new net c2: SW13.1, SW14.1, SW15.1, SW16.1, SW17.1, SW18.1, U1.3 (GPB2)
- new net c3: SW19.1, SW20.1, SW21.1, SW22.1, SW23.1, SW24.1, U1.4 (GPB3)
- new net c4: SW25.1, SW26.1, SW27.1, SW28.1, SW29.1, SW30.1, U1.5 (GPB4)
- new net c5: SW31.1, SW32.1, SW33.1, SW34.1, SW35.1, SW36.1, U1.6 (GPB5)
- new net c6: SW37.1, SW38.1, SW39.1, SW40.1, SW41.1, SW42.1, U1.7 (GPB6)
- new net c7: SW43.1, SW44.1, SW45.1, SW46.1, SW47.1, SW48.1, U1.21 (GPA0)
- new net c8: SW49.1, SW50.1, SW51.1, SW52.1, SW53.1, SW54.1, U1.22 (GPA1)
- new net c9: SW55.1, SW56.1, SW57.1, SW58.1, SW59.1, SW60.1, U1.23 (GPA2)
- new net r0: D1.1 (K), D13.1 (K), D19.1 (K), D25.1 (K), D31.1 (K), D37.1 (K), D43.1 (K), D49.1 (K), D55.1 (K), D61.1 (K), D66.1 (K), D7.1 (K), D71.1 (K), D75.1 (K), U2.3 (D5)
- new net r1: D14.1 (K), D2.1 (K), D20.1 (K), D26.1 (K), D32.1 (K), D38.1 (K), D44.1 (K), D50.1 (K), D56.1 (K), D62.1 (K), D67.1 (K), D72.1 (K), D76.1 (K), D8.1 (K), U2.4 (D6)
- new net r2: D15.1 (K), D21.1 (K), D27.1 (K), D3.1 (K), D33.1 (K), D39.1 (K), D45.1 (K), D51.1 (K), D57.1 (K), D63.1 (K), D68.1 (K), D73.1 (K), D77.1 (K), D9.1 (K), U2.5 (D9)
- new net r3: D10.1 (K), D16.1 (K), D22.1 (K), D28.1 (K), D34.1 (K), D4.1 (K), D40.1 (K), D46.1 (K), D52.1 (K), D58.1 (K), D64.1 (K), D69.1 (K), D74.1 (K), U2.6 (D10)
- new net r4: D11.1 (K), D17.1 (K), D23.1 (K), D29.1 (K), D35.1 (K), D41.1 (K), D47.1 (K), D5.1 (K), D53.1 (K), D59.1 (K), D65.1 (K), D70.1 (K), U2.7 (D11)
- new net r5: D12.1 (K), D18.1 (K), D24.1 (K), D30.1 (K), D36.1 (K), D42.1 (K), D48.1 (K), D54.1 (K), D6.1 (K), D60.1 (K), U2.8 (D12)
- no-connect marks 1 -> 0
